File: MCU_Node_V1/MCU_Node_V1.kicad_sch (KiCad schematic)
At the start: 88 parts, among them J1 Conn_01x02_Socket, J10 Conn_01x02_Socket, J11 USB_B_Micro, J12 POWER_SELECT, J13 Conn_01x02_Socket, J14 Conn_01x02_Socket, J15 Conn_01x02_Socket, J16 Conn_01x02_Socket, J17 Conn_01x02_Socket, J18 Conn_01x02_Socket, J2 DC_IN, J3 Conn_01x03_Socket, J4 Timer Config, J5 LPM_BYP, J6 Conn_01x08, J7 Conn_01x08, J8 Conn_01x14, J9 REG_EN, Q1 BSS138, Q3 PMOS, Q4 BSS138, SW1 SW_Push, SW2 SW_Push, SW3 LPM_RST, U1 74HC595, U2 CH340C, U5 ESP32-WROOM-32, U6 TPL5110, U7 AMS1117-3.3

Commit message: edit
edited mikroe symbol & footprint
edited extra pinouts
added solder jumper 74HC595
added mounting hole
Parts:
- removed J6, J7: Conn_01x08, Connector_PinHeader_2.54mm:PinHeader_1x08_P2.54mm_Vertical, symbol Connector_Generic:Conn_01x08
- removed J8: Conn_01x14, symbol Connector_Generic:Conn_01x14
- added H1, H2, H3: MountingHole, MountingHole:MountingHole_3.2mm_M3_DIN965_Pad, symbol Mechanical:MountingHole
- added J6: Conn_01x10, Connector_PinHeader_2.54mm:PinHeader_1x10_P2.54mm_Vertical, symbol Connector_Generic:Conn_01x10
- added J7, J8: Conn_01x02, Connector_PinHeader_2.54mm:PinHeader_1x02_P2.54mm_Vertical, symbol Connector_Generic:Conn_01x02
- added JP13, JP14, JP15: SolderJumper_2_Open, Jumper:SolderJumper-2_P1.3mm_Open_Pad1.0x1.5mm, symbol Jumper:SolderJumper_2_Open
- added U3: MIKROE, MIKROE_3800:MIKROE-3800, symbol MIKROE-3800:MIKROE-3800
- J1, J10, J13, J14, J15, J16, J17, J18: footprint (none) -> Connector_PinHeader_2.54mm:PinHeader_1x02_P2.54mm_Vertical
Connections:
- net +3.3V: now also J8.2 (Pin_2), U3.7 (+3.3V)
- net GND: now also J7.1 (Pin_1), J8.1 (Pin_1), U3.8 (GND), U3.9 (GND2)
- net IO_14: now also J6.6 (Pin_6)
- net IO_2: now also J6.4 (Pin_4)
- net IO_25: now also J6.3 (Pin_3), JP13.1 (A); no longer U1.14 (SER)
- net IO_26: now also J6.2 (Pin_2), JP14.1 (A); no longer U1.11 (SRCLK)
- net IO_27: now also J6.1 (Pin_1), JP15.1 (A); no longer U1.12 (RCLK)
- net IO_34: now also J6.7 (Pin_7)
- net IO_35: now also J6.8 (Pin_8)
- net IO_4: now also J6.5 (Pin_5)
- net MIKROE_AIN: now also U3.1 (AIN)
- net MIKROE_CS: now also U3.3 (CS)
- net MIKROE_INT: now also U3.15 (INT)
- net MIKROE_PWM: now also U3.16 (PWM)
- net MIKROE_RST: now also U3.2 (RST)
- net MIKROE_RX: now also U3.13 (RX)
- net MIKROE_SCK: now also U3.4 (SCK)
- net MIKROE_SCL: now also J6.10 (Pin_10), U3.12 (SCL)
- net MIKROE_SDA: now also J6.9 (Pin_9), U3.11 (SDA)
- net MIKROE_SDI: now also U3.6 (SDI)
- net MIKROE_SDO: now also U3.5 (SDO)
- net MIKROE_TX: now also U3.14 (TX)
- net VCC: now also J7.2 (Pin_2), U3.10 (5V)
- new net: JP14.2 (B), U1.11 (SRCLK)
- new net: JP15.2 (B), U1.12 (RCLK)
- new net: JP13.2 (B), U1.14 (SER)
Other:
- note added: "EXTERNAL OUTPUT SUPPLY"

Commit message: -
Parts:
- added H4: MountingHole, MountingHole:MountingHole_3.2mm_M3_DIN965_Pad, symbol Mechanical:MountingHole
Changed lines of the file:
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@@
+	)
+	(symbol
+		(lib_id "Mechanical:MountingHole")
+		(at 39.3739 306.3016 0)
+		(unit 1)
+		(exclude_from_sim yes)
+		(in_bom no)
+		(on_board yes)
+		(dnp no)
+		(fields_autoplaced yes)
+		(property "Reference" "H4"
+			(at 42.1023 305.0315 0)
+			(effects
+				(font
+					(size 1.27 1.27)
+				)
+				(justify left)
+			)
+		)
+		(property "Value" "MountingHole"
+			(at 42.1023 307.5715 0)
+			(effects
+				(font
+					(size 1.27 1.27)
+				)
+				(justify left)
+			)
+		)
+		(property "Footprint" "MountingHole:MountingHole_3.2mm_M3_DIN965_Pad"
+			(at 39.3739 306.3016 0)
+			(effects
+				(font
+					(size 1.27 1.27)
+				)
+				(hide yes)
+			)
+		)
+		(property "Datasheet" "~"
+			(at 39.3739 306.3016 0)
+			(effects
+				(font
+					(size 1.27 1.27)
+				)
+				(hide yes)
+			)
+		)
+		(property "Description" "Mounting Hole without connection"
+			(at 39.3739 306.3016 0)
+			(effects
+				(font
+					(size 1.27 1.27)
+				)
+				(hide yes)
+			)
+		)
+		(instances
+			(project "MCU_Node_V1"
+				(path "/8f3fcdef-c1c5-4633-bb68-bb9798a055e2"
+					(reference "H4")
+					(unit 1)
+				)
+			)
+		)
 	)
 	(symbol
