File: MCU_Node_V1/MCU_Node_V1.kicad_sch (KiCad schematic)
At the start: 122 parts, among them J1 Conn_01x02_Socket, J10 Conn_01x02_Socket, J11 USB_B_Micro, J12 POWER_SELECT, J13 Conn_01x02_Socket, J14 Conn_01x02_Socket, J15 Conn_01x02_Socket, J16 Conn_01x02_Socket, J17 Conn_01x02_Socket, J18 Conn_01x02_Socket, J19 Timer Config, J2 DC_IN, J20 LPM_BYP, J3 Conn_01x03_Socket, J4 Timer Config, J5 LPM_BYP, J6 Conn_01x10, J7 Conn_01x02, J8 Conn_01x02, J9 REG_EN, Q1 BSS138, Q3 PMOS, Q4 BSS138, SW1 SW_Push, SW2 SW_Push, SW3 LPM_RST, SW4 LPM_RST, U1 74HC595, U2 CH340C, U3 MIKROE, U4 TPS73733DCQR, U5 ESP32-WROOM-32, U6 TPL5110, U7 AMS1117-3.3, U8 TPL5110

Commit message: Update Saved Files for  3V3 Regulator change
Parts:
- removed C10, C11, C13: 0.1uF, Capacitor_SMD:C_0402_1005Metric, symbol Device:C
- removed C12, C14: 10uF, Capacitor_SMD:C_0805_2012Metric_Pad1.18x1.45mm_HandSolder, symbol Device:C
- removed D11: LED, LED_SMD:LED_0805_2012Metric_Pad1.15x1.40mm_HandSolder, symbol Device:LED
- removed J20, J5: LPM_BYP, Connector_PinHeader_2.54mm:PinHeader_1x02_P2.54mm_Vertical, symbol Connector_Generic:Conn_01x02
- removed J4: Timer Config, Connector_IDC:IDC-Header_2x08_P2.54mm_Vertical, symbol Connector_Generic:Conn_02x08_Odd_Even
- removed JP1: SolderJumper_3_Open, Jumper:SolderJumper-3_P1.3mm_Open_Pad1.0x1.5mm, symbol Jumper:SolderJumper_3_Open
- removed JP12, JP2: SolderJumper_2_Open, Jumper:SolderJumper-2_P1.3mm_Open_Pad1.0x1.5mm, symbol Jumper:SolderJumper_2_Open
- removed Q3: PMOS, Package_TO_SOT_SMD:SOT-23-3, symbol Simulation_SPICE:PMOS
- removed R10: 169K, Resistor_SMD:R_0603_1608Metric_Pad0.98x0.95mm_HandSolder, symbol Device:R
- removed R11: 124K, Resistor_SMD:R_0603_1608Metric_Pad0.98x0.95mm_HandSolder, symbol Device:R
- removed R12: 91K, Resistor_SMD:R_0603_1608Metric_Pad0.98x0.95mm_HandSolder, symbol Device:R
- removed R13: 76.8K, Resistor_SMD:R_0603_1608Metric_Pad0.98x0.95mm_HandSolder, symbol Device:R
- removed R14: 16.9K, Resistor_SMD:R_0603_1608Metric_Pad0.98x0.95mm_HandSolder, symbol Device:R
- removed R21: 1K, Resistor_SMD:R_0603_1608Metric_Pad0.98x0.95mm_HandSolder, symbol Device:R
- removed R6: 1M, Resistor_SMD:R_0603_1608Metric_Pad0.98x0.95mm_HandSolder, symbol Device:R
- removed R7: 22K, Resistor_SMD:R_0603_1608Metric_Pad0.98x0.95mm_HandSolder, symbol Device:R
- removed R8: 43.2K, Resistor_SMD:R_0603_1608Metric_Pad0.98x0.95mm_HandSolder, symbol Device:R
- removed R9: 34.8K, Resistor_SMD:R_0603_1608Metric_Pad0.98x0.95mm_HandSolder, symbol Device:R
- removed SW3: LPM_RST, Button_Switch_SMD:SW_SPST_CK_RS282G05A3, symbol Switch:SW_Push
- removed U6: TPL5110, Package_TO_SOT_SMD:SOT-23-6, symbol Timer:TPL5110
- removed U7: AMS1117-3.3, Package_TO_SOT_SMD:SOT-223-3_TabPin2, symbol Regulator_Linear:AMS1117-3.3
- added J4: REG_CTRL, Connector_PinHeader_2.54mm:PinHeader_1x03_P2.54mm_Vertical, symbol Connector_Generic:Conn_01x03
Connections:
- net GND: now also J4.1 (Pin_1)
- net VCC: now also J4.3 (Pin_3)
- net at JP17.1 (A), R31.2, U4.5 (EN): now also J4.2 (Pin_2)
Other:
- moved on the sheet: C16, C17, C18, C19, C20, C21, D12, H1, H2, H3, H4, J19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
