File: MCU_Node_V1/MCU_Node_V1.kicad_pcb (KiCad board)
At the start: 2 copper layers, 100.6 x 40.1 mm, 97 parts, among them J1 Conn_01x02_Socket, J10 Conn_01x02_Socket, J11 USB_B_Micro, J12 POWER_SELECT, J13 Conn_01x02_Socket, J14 Conn_01x02_Socket, J15 Conn_01x02_Socket, J16 Conn_01x02_Socket, J17 Conn_01x02_Socket, J18 Conn_01x02_Socket, J19 Timer Config, J2 DC_IN, J3 Conn_01x03_Socket, J4 REG_CTRL, J6 Conn_01x10, J7 Conn_01x02, J8 Conn_01x02, J9 REG_EN, Q1 BSS138, Q4 BSS138, SW1 SW_Push, SW2 SW_Push, SW4 LPM_RST, U1 74HC595, U2 CH340C, U3 MIKROE, U4 TPS73733DCQR, U5 ESP32-WROOM-32, U8 TPL5110

Commit message: -
routing & placement done
Parts:
- J19: footprint Connector_PinHeader_2.54mm:PinHeader_2x08_P2.54mm_Vertical -> Connector_IDC:IDC-Header_2x08_P2.54mm_Vertical
- JP10, JP11, JP13, JP14, JP15, JP3, JP4, JP5, JP6, JP7, JP8, JP9: moved to B.Cu
- moved J9 121.5 mm to (232.8, 55.0)
- moved R5 110.1 mm to (177.4, 63.3), turned to 180 degrees
- moved C7 98.6 mm to (175.4, 85.0), turned to 180 degrees
- moved C6 97.6 mm to (175.3, 86.7), turned to 180 degrees
- moved C8 94.8 mm to (180.5, 62.0)
- moved C4 92.9 mm to (176.0, 62.0), turned to 180 degrees
- moved C5 91.4 mm to (174.7, 63.4)
- moved C2 73.4 mm to (197.1, 74.3)
- moved C15 64.6 mm to (197.7, 75.9)
- moved JP11 63.8 mm to (208.4, 84.0), turned to 180 degrees
- moved JP13 54.7 mm to (191.9, 83.8), turned to 90 degrees
- moved JP7 50.8 mm to (191.3, 92.5), turned to 90 degrees
- moved JP10 49.1 mm to (199.0, 92.6), turned to 90 degrees
- moved JP15 47.4 mm to (197.1, 83.8), turned to 90 degrees
- moved JP6 46.6 mm to (188.7, 92.5), turned to 90 degrees
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Routing:
- net MIKROE_3V3: track 1.44 -> 123.7 mm, vias 1 -> 9
- net MIKROE_SCL: track 0.00 -> 99.3 mm, vias 0 -> 2
- net MIKROE_SDO: track 0.00 -> 94.0 mm, vias 0 -> 2
- net MIKROE_SDA: track 0.00 -> 93.6 mm, vias 0 -> 2
- net MIKROE_SDI: track 0.00 -> 86.5 mm, vias 0 -> 2
- net IO_2: track 0.00 -> 86.0 mm, vias 0 -> 2
- net IO_4: track 0.00 -> 82.4 mm, vias 0 -> 2
- net IO_25: track 0.00 -> 82.2 mm, vias 0 -> 2
- net MIKROE_SCK: track 0.00 -> 80.7 mm, vias 0 -> 2
- net IO_34: track 0.00 -> 79.7 mm, vias 0 -> 2
- net IO_35: track 0.00 -> 78.9 mm, vias 0 -> 2
- net MIKROE_CS: track 0.00 -> 77.1 mm, vias 0 -> 2
- net IO_26: track 0.00 -> 75.0 mm, vias 0 -> 1
- net IO_27: track 0.00 -> 73.4 mm, vias 0 -> 1
- net IO_14: track 0.00 -> 72.7 mm, vias 0 -> 2
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- added copper zone on F.Cu, net ESP_EN
- added copper zone on B.Cu, net MIKROE_3V3
- added copper zone on B.Cu, net MIKROE_GND
- added copper zone on F.Cu, net MIKROE_GND
Other:
- board size 100.6 x 40.1 mm -> 90.2 x 48.8 mm

Commit message: -
Parts:
- moved U4 4.10 mm to (214.7, 67.6)
- moved J1 3.95 mm to (176.7, 98.3)
- moved J10 3.06 mm to (180.3, 98.3)
- moved J18 2.27 mm to (202.4, 98.3)
- moved J13 2.18 mm to (184.0, 98.3)
- moved J17 1.38 mm to (198.8, 98.3)
- moved J14 1.29 mm to (187.7, 98.3)
- moved U1 0.85 mm to (202.6, 79.4)
- moved C15 0.84 mm to (197.7, 75.0)
- moved C2 0.81 mm to (197.2, 73.5)
- moved J8 0.81 mm to (247.5, 98.3)
- moved J7 0.75 mm to (247.5, 53.3)
- moved H2 0.50 mm to (169.7, 96.8)
- moved J16 0.49 mm to (195.1, 98.3)
- moved H3 0.45 mm to (253.2, 96.8)
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Routing:
- net MIKROE_GND: track 61.7 -> 71.7 mm, vias 67 -> 154
- net Net-(J10-Pin_2): track 30.8 -> 35.9 mm
- net MIKROE_5V: track 59.3 -> 64.3 mm
- net Net-(J1-Pin_2): track 37.2 -> 41.4 mm
- net Net-(J4-Pin_2): track 38.7 -> 42.8 mm
- net Net-(U4-FB): track 2.04 -> 6.15 mm
- net Net-(J13-Pin_2): track 28.3 -> 31.1 mm
- net Net-(J18-Pin_2): track 18.5 -> 20.7 mm
- net MIKROE_3V3: track 123.7 -> 121.7 mm
- net Net-(J14-Pin_2): track 26.5 -> 28.2 mm
- net Net-(JP14-B): track 17.0 -> 18.2 mm
- net Net-(JP11-B): track 4.10 -> 4.95 mm
- net Net-(J15-Pin_2): track 24.0 -> 24.9 mm
- net Net-(JP13-B): track 11.7 -> 12.2 mm
Other:
- board text added: "*"
- board text added: "+"
- board text added: "-"
- board text added: "ESP_RX"
- board text added: "ESP_TX"
- board text added: "GND"
